File: pcb/plotter/plotter.kicad_pcb (KiCad board)
At the start: 2 copper layers, 222.6 x 42.4 mm, 80 parts, among them J1 SH 1106 Display, J10 Limit switches, J2 SWD, J3 Console, J4 Micro_SD_Card_Det, J5 USB_B_Micro, J6 Barrel_Jack_Switch, J8 Motor2, J9 Motor1, SW1 Rotary_Encoder_Switch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

Commit message: Schematics minor changes
Parts:
- C1: value CP -> 22µF 16V
- C29, C35: value CP -> 100µF
- R12: value 22R -> 1k
- turned C29 to 0 degrees
- turned C35 to 0 degrees
Connections:
- net Net-(J1-Pad1) renamed /sda
- net Net-(J1-Pad2) renamed /scl
- C29 pad 1: GND -> +24V
- C29 pad 2: +24V -> GND
- C35 pad 1: GND -> +24V
- C35 pad 2: +24V -> GND
Changed lines of the file:
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@@
   (net 21 "Net-(C21-Pad1)")
   (net 22 "+24V")
-  (net 23 "Net-(J1-Pad1)")
-  (net 24 "Net-(J1-Pad2)")
+  (net 23 "/sda")
+  (net 24 "/scl")
   (net 25 "Net-(J3-Pad1)")
   (net 26 "unconnected-(U2-Pad14)")
@@
     (property "Sheetname" "Motors")
     (attr smd)
-    (fp_text reference "C32" (at -0.444 1.424 180) (layer "F.SilkS")
+    (fp_text reference "C32" (at -0.014 1.284 180) (layer "F.SilkS")
       (effects (font (size 0.635 0.635) (thickness 0.1016)))
     )
@@
   )
   (footprint "Capacitor_SMD:CP_Elec_8x10" (layer "F.Cu")
-    (at 105.156 93.41 180)
+    (at 105.156 93.41)
     (descr "SMD capacitor, aluminum electrolytic, Nichicon, 8.0x10mm")
     (tags "capacitor electrolytic")
@@
     (property "Sheetname" "Motors")
     (attr smd)
-    (fp_text reference "C29" (at -5.244 -3.59 180) (layer "F.SilkS")
+    (fp_text reference "C29" (at -4.466 -4.56) (layer "F.SilkS")
       (effects (font (size 0.635 0.635) (thickness 0.1016)))
     )
-    (fp_text value "CP" (at 0 5.2) (layer "F.Fab")
+    (fp_text value "100µF" (at 0 5.2) (layer "F.Fab")
       (effects (font (size 0.635 0.635) (thickness 0.1016)))
     )
@@
     (fp_line (start -4.15 -3.15) (end -3.15 -4.15) (layer "F.Fab") (width 0.1))
     (fp_circle (center 0 0) (end 4 0) (layer "F.Fab") (width 0.1) (fill none))
-    (pad "1" smd roundrect locked (at -3.25 0 180) (size 3.5 2.5) (layers "F.Cu" "F.Paste" "F.Mask") (roundrect_rratio 0.1)
-      (net 44 "GND") (pintype "passive"))
-    (pad "2" smd roundrect locked (at 3.25 0 180) (size 3.5 2.5) (layers "F.Cu" "F.Paste" "F.Mask") (roundrect_rratio 0.1)
+    (pad "1" smd roundrect locked (at -3.25 0) (size 3.5 2.5) (layers "F.Cu" "F.Paste" "F.Mask") (roundrect_rratio 0.1)
       (net 22 "+24V") (pintype "passive"))
+    (pad "2" smd roundrect locked (at 3.25 0) (size 3.5 2.5) (layers "F.Cu" "F.Paste" "F.Mask") (roundrect_rratio 0.1)
+      (net 44 "GND") (pintype "passive"))
     (model "${KISYS3DMOD}/Capacitor_SMD.3dshapes/CP_Elec_8x10.wrl"
       (offset (xyz 0 0 0))
@@
     (fp_line (start 5.09 -14.74) (end 5.09 -12.2) (layer "F.Fab") (width 0.1))
     (pad "1" thru_hole rect locked (at -3.8 -13.47 180) (size 1.7 1.7) (drill 1) (layers *.Cu *.Mask)
-      (net 23 "Net-(J1-Pad1)") (pinfunction "Pin_1") (pintype "passive"))
+      (net 23 "/sda") (pinfunction "Pin_1") (pintype "passive"))
     (pad "2" thru_hole oval locked (at -1.26 -13.47 180) (size 1.7 1.7) (drill 1) (layers *.Cu *.Mask)
-      (net 24 "Net-(J1-Pad2)") (pinfunction "Pin_2") (pintype "passive"))
+      (net 24 "/scl") (pinfunction "Pin_2") (pintype "passive"))
     (pad "3" thru_hole oval locked (at 1.28 -13.47 180) (size 1.7 1.7) (drill 1) (layers *.Cu *.Mask)
       (net 44 "GND") (pinfunction "Pin_3") (pintype "passive"))
@@
       (effects (font (size 0.635 0.635) (thickness 0.1016)))
     )
-    (fp_text value "CP" (at 0 5.2) (layer "F.Fab")
+    (fp_text value "22µF 16V" (at 0 5.2) (layer "F.Fab")
       (effects (font (size 0.635 0.635) (thickness 0.1016)))
     )
@@
   )
   (footprint "Capacitor_SMD:CP_Elec_8x10" (layer "F.Cu")
-    (at 105.156 110.2 180)
+    (at 105.156 110.2)
     (descr "SMD capacitor, aluminum electrolytic, Nichicon, 8.0x10mm")
     (tags "capacitor electrolytic")
@@
     (property "Sheetname" "Motors")
     (attr smd)
-    (fp_text reference "C35" (at -5.244 -3.8) (layer "F.SilkS")
+    (fp_text reference "C35" (at 4.954 -3.44 90) (layer "F.SilkS")
       (effects (font (size 0.635 0.635) (thickness 0.1016)))
     )
-    (fp_text value "CP" (at 0 5.2) (layer "F.Fab")
+    (fp_text value "100µF" (at 0 5.2) (layer "F.Fab")
       (effects (font (size 0.635 0.635) (thickness 0.1016)))
     )
@@
     (fp_line (start -4.15 -3.15) (end -4.15 3.15) (layer "F.Fab") (width 0.1))
     (fp_circle (center 0 0) (end 4 0) (layer "F.Fab") (width 0.1) (fill none))
-    (pad "1" smd roundrect locked (at -3.25 0 180) (size 3.5 2.5) (layers "F.Cu" "F.Paste" "F.Mask") (roundrect_rratio 0.1)
-      (net 44 "GND") (pintype "passive"))
-    (pad "2" smd roundrect locked (at 3.25 0 180) (size 3.5 2.5) (layers "F.Cu" "F.Paste" "F.Mask") (roundrect_rratio 0.1)
+    (pad "1" smd roundrect locked (at -3.25 0) (size 3.5 2.5) (layers "F.Cu" "F.Paste" "F.Mask") (roundrect_rratio 0.1)
       (net 22 "+24V") (pintype "passive"))
+    (pad "2" smd roundrect locked (at 3.25 0) (size 3.5 2.5) (layers "F.Cu" "F.Paste" "F.Mask") (roundrect_rratio 0.1)
+      (net 44 "GND") (pintype "passive"))
     (model "${KISYS3DMOD}/Capacitor_SMD.3dshapes/CP_Elec_8x10.wrl"
       (offset (xyz 0 0 0))
@@
       (net 68 "/dir1") (pinfunction "PB5") (pintype "bidirectional"))
     (pad "58" smd roundrect locked (at -0.75 -5.675 90) (size 0.3 1.55) (layers "F.Cu" "F.Paste" "F.Mask") (roundrect_rratio 0.25)
-      (net 24 "Net-(J1-Pad2)") (pinfunction "PB6") (pintype "bidirectional"))
+      (net 24 "/scl") (pinfunction "PB6") (pintype "bidirectional"))
     (pad "59" smd roundrect locked (at -1.25 -5.675 90) (size 0.3 1.55) (layers "F.Cu" "F.Paste" "F.Mask") (roundrect_rratio 0.25)
-      (net 23 "Net-(J1-Pad1)") (pinfunction "PB7") (pintype "bidirectional"))
+      (net 23 "/sda") (pinfunction "PB7") (pintype "bidirectional"))
     (pad "60" smd roundrect locked (at -1.75 -5.675 90) (size 0.3 1.55) (layers "F.Cu" "F.Paste" "F.Mask") (roundrect_rratio 0.25)
       (net 3 "Net-(R12-Pad2)") (pinfunction "BOOT0") (pintype "input"))
@@
       (effects (font (size 0.635 0.635) (thickness 0.1016)))
     )
-    (fp_text value "22R" (at 0 1.43) (layer "F.Fab")
+    (fp_text value "1k" (at 0 1.43) (layer "F.Fab")
       (effects (font (size 0.635 0.635) (thickness 0.1016)))
     )
