File: pcb/plotter/plotter.kicad_sch (KiCad schematic)
At the start: 57 parts, among them J1 SH 1106 Display, J10 Limit switches, J2 SWD, J3 Console, J4 Micro_SD_Card_Det, J5 USB_B_Micro, SW1 Rotary_Encoder_Switch, U1 STM32F405RGTx, U4 PUSB3F96, U6 AP1117-33, U7 PUSB3F96, U8 PUSB3F96

Commit message: I finally got the SD card to work.
Parts:
- added R13: 10k, Resistor_SMD:R_0603_1608Metric, symbol Device:R
Connections:
- net VDD: now also R13.1
- net sdMosi: now reaches J4.3 (CMD), U7.4
- net sdMosi: now also U1.53 (PC12); no longer U1.23 (PA7)
- net sdSck: now reaches J4.5 (CLK), U7.2
- net sdSck: now also U1.51 (PC10); no longer U1.21 (PA5)
- net sdMiso: now reaches J4.7 (DAT0), U7.1
- net sdMiso: now also U1.52 (PC11), R13.2; no longer U1.22 (PA6)
Changed lines of the file:
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@@
   (junction (at 212.725 54.61) (diameter 1.016) (color 0 0 0 0))
   (junction (at 215.265 57.15) (diameter 1.016) (color 0 0 0 0))
+  (junction (at 215.265 64.77) (diameter 1.016) (color 0 0 0 0))
   (junction (at 225.425 88.9) (diameter 1.016) (color 0 0 0 0))
   (junction (at 227.965 83.82) (diameter 1.016) (color 0 0 0 0))
@@
   (no_connect (at 139.065 121.92))
   (no_connect (at 139.065 124.46))
-  (no_connect (at 139.065 127))
-  (no_connect (at 139.065 129.54))
-  (no_connect (at 139.065 132.08))
+  (no_connect (at 174.625 71.12))
+  (no_connect (at 174.625 73.66))
+  (no_connect (at 174.625 76.2))
   (no_connect (at 174.625 78.74))
   (no_connect (at 174.625 81.28))
@@
     (stroke (width 0) (type solid) (color 0 0 0 0))
   )
-  (wire (pts (xy 174.625 71.12) (xy 212.725 71.12))
-    (stroke (width 0) (type solid) (color 0 0 0 0))
-  )
-  (wire (pts (xy 174.625 73.66) (xy 215.265 73.66))
-    (stroke (width 0) (type solid) (color 0 0 0 0))
-  )
-  (wire (pts (xy 174.625 76.2) (xy 210.185 76.2))
-    (stroke (width 0) (type solid) (color 0 0 0 0))
-  )
   (wire (pts (xy 174.625 88.9) (xy 208.915 88.9))
     (stroke (width 0) (type solid) (color 0 0 0 0))
@@
     (stroke (width 0) (type solid) (color 0 0 0 0))
   )
+  (wire (pts (xy 184.15 76.2) (xy 210.185 76.2))
+    (stroke (width 0) (type solid) (color 0 0 0 0))
+  )
+  (wire (pts (xy 184.785 73.66) (xy 215.265 73.66))
+    (stroke (width 0) (type solid) (color 0 0 0 0))
+  )
+  (wire (pts (xy 185.42 71.12) (xy 212.725 71.12))
+    (stroke (width 0) (type solid) (color 0 0 0 0))
+  )
   (wire (pts (xy 186.69 52.07) (xy 187.325 52.07))
     (stroke (width 0) (type solid) (color 0 0 0 0))
@@
     (stroke (width 0) (type solid) (color 0 0 0 0))
   )
-  (wire (pts (xy 215.265 57.15) (xy 215.265 73.66))
+  (wire (pts (xy 215.265 57.15) (xy 215.265 64.77))
+    (stroke (width 0) (type solid) (color 0 0 0 0))
+  )
+  (wire (pts (xy 215.265 64.77) (xy 215.265 73.66))
+    (stroke (width 0) (type solid) (color 0 0 0 0))
+  )
+  (wire (pts (xy 215.265 64.77) (xy 217.805 64.77))
     (stroke (width 0) (type solid) (color 0 0 0 0))
   )
@@
     (effects (font (size 1.27 1.27)) (justify right bottom))
   )
+  (label "sdSck" (at 139.065 127 180)
+    (effects (font (size 1.27 1.27)) (justify right bottom))
+  )
+  (label "sdMiso" (at 139.065 129.54 180)
+    (effects (font (size 1.27 1.27)) (justify right bottom))
+  )
+  (label "sdMosi" (at 139.065 132.08 180)
+    (effects (font (size 1.27 1.27)) (justify right bottom))
+  )
   (label "dir2" (at 139.065 134.62 180)
     (effects (font (size 1.27 1.27)) (justify right bottom))
@@
     (effects (font (size 1.27 1.27)) (justify left bottom))
   )
+  (label "sdMosi" (at 184.15 76.2 180)
+    (effects (font (size 1.27 1.27)) (justify right bottom))
+  )
+  (label "sdMiso" (at 184.785 73.66 180)
+    (effects (font (size 1.27 1.27)) (justify right bottom))
+  )
+  (label "sdSck" (at 185.42 71.12 180)
+    (effects (font (size 1.27 1.27)) (justify right bottom))
+  )
   (label "esd1" (at 220.98 55.88 270)
     (effects (font (size 1.27 1.27)) (justify right bottom))
@@
     )
     (property "Datasheet" "" (id 3) (at 203.835 29.21 0)
+      (effects (font (size 1.27 1.27)) hide)
+    )
+    (pin "1")
+  )
+  (symbol (lib_id "power:VDD") (at 217.805 72.39 180) (unit 1)
+    (in_bom yes) (on_board yes) (fields_autoplaced)
+    (property "Reference" "#PWR0129" (id 0) (at 217.805 68.58 0)
+      (effects (font (size 1.27 1.27)) hide)
+    )
+    (property "Value" "VDD" (id 1) (at 219.2021 73.9485 0)
+      (effects (font (size 1.27 1.27)) (justify right))
+    )
+    (property "Footprint" "" (id 2) (at 217.805 72.39 0)
+      (effects (font (size 1.27 1.27)) hide)
+    )
+    (property "Datasheet" "" (id 3) (at 217.805 72.39 0)
       (effects (font (size 1.27 1.27)) hide)
     )
@@
     )
     (property "Datasheet" "~" (id 3) (at 212.725 106.045 0)
+      (effects (font (size 1.27 1.27)) hide)
+    )
+    (pin "1")
+    (pin "2")
+  )
+  (symbol (lib_id "Device:R") (at 217.805 68.58 180) (unit 1)
+    (in_bom yes) (on_board yes) (fields_autoplaced)
+    (property "Reference" "R13" (id 0) (at 219.5831 67.6715 0)
+      (effects (font (size 1.27 1.27)) (justify right))
+    )
+    (property "Value" "10k" (id 1) (at 219.5831 70.4466 0)
+      (effects (font (size 1.27 1.27)) (justify right))
+    )
+    (property "Footprint" "Resistor_SMD:R_0603_1608Metric" (id 2) (at 219.583 68.58 90)
+      (effects (font (size 1.27 1.27)) hide)
+    )
+    (property "Datasheet" "~" (id 3) (at 217.805 68.58 0)
       (effects (font (size 1.27 1.27)) hide)
     )
@@
       (reference "#PWR0128") (unit 1) (value "GND") (footprint "")
     )
+    (path "/40806812-3b09-4dac-99ed-960a83e904ed"
+      (reference "#PWR0129") (unit 1) (value "VDD") (footprint "")
+    )
     (path "/c73a8afd-1bb2-4582-b865-0602b4353a4c"
       (reference "C1") (unit 1) (value "CP") (footprint "Capacitor_SMD:CP_Elec_8x10")
@@
       (reference "R12") (unit 1) (value "22R") (footprint "Resistor_SMD:R_0603_1608Metric")
     )
+    (path "/eeb70e44-13ce-434f-85a7-b1797c59da79"
+      (reference "R13") (unit 1) (value "10k") (footprint "Resistor_SMD:R_0603_1608Metric")
+    )
     (path "/aad9a816-7f7b-42ba-adfd-b21451a17f15"

Commit message: Bringing up the first PCB
Parts:
- C1: value CP -> 22µF 16V
- R12: value 22R -> 1k
Connections:
- net sda: now reaches J1.1 (Pin_1), U1.59 (PB7)
- net scl: now reaches J1.2 (Pin_2), U1.58 (PB6)
Other:
- note added: "TODO : SWD header has some crazy pitch like 1.25. Change Console header has 3 pins instead of 4 (same component) Increase 100µF Electrolityc Capacaitors footprints to maximum available (that fits). SWitch to the most popular micro sd holder footprint. Now im stuck as there is no parts with the footprint i've chosen. OLED display footprint has wrong pin order (mirrored). SWD header is pretty bad p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"
Changed lines of the file:
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@@
     (effects (font (size 1.27 1.27)) (justify right bottom))
+  )
+  (text "TODO : SWD header has some crazy pitch like 1.25. Change\nConsole header has 3 pins instead of 4 (same component)\nIncrease 100µF Electrolityc Capacaitors footprints to maximum available (that fits).\nSWitch to the most popular micro sd holder footprint. Now im stuck as there is no parts with the footprint i've chosen.\nOLED display footprint has wrong pin order (mirrored).\nSWD header is pretty bad placed. The cable attached gets tangled ."
+    (at 129.54 -10.795 0)
+    (effects (font (size 1.27 1.27)) (justify left bottom))
   )
   (label "servo" (at 42.545 179.07 0)
@@
   (label "sdSck" (at 185.42 71.12 180)
     (effects (font (size 1.27 1.27)) (justify right bottom))
+  )
+  (label "scl" (at 189.23 116.84 0)
+    (effects (font (size 1.27 1.27)) (justify left bottom))
+  )
+  (label "sda" (at 194.31 119.38 0)
+    (effects (font (size 1.27 1.27)) (justify left bottom))
   )
   (label "esd1" (at 220.98 55.88 270)
@@
     (in_bom yes) (on_board yes) (fields_autoplaced)
     (property "Reference" "R12" (id 0) (at 132.08 58.5174 90))
-    (property "Value" "22R" (id 1) (at 132.08 61.2925 90))
+    (property "Value" "1k" (id 1) (at 132.08 61.2925 90))
     (property "Footprint" "Resistor_SMD:R_0603_1608Metric" (id 2) (at 132.08 65.278 90)
       (effects (font (size 1.27 1.27)) hide)
@@
   (symbol (lib_id "Device:CP") (at 43.815 186.055 0) (mirror y) (unit 1)
     (in_bom yes) (on_board yes) (fields_autoplaced)
-    (property "Reference" "C1" (id 0) (at 46.7361 186.9635 0)
-      (effects (font (size 1.27 1.27)) (justify right))
-    )
-    (property "Value" "CP" (id 1) (at 46.7361 184.1884 0)
+    (property "Reference" "C1" (id 0) (at 46.7361 185.1465 0)
+      (effects (font (size 1.27 1.27)) (justify right))
+    )
+    (property "Value" "22µF 16V" (id 1) (at 46.7361 187.9216 0)
       (effects (font (size 1.27 1.27)) (justify right))
     )
@@
     )
     (path "/c73a8afd-1bb2-4582-b865-0602b4353a4c"
-      (reference "C1") (unit 1) (value "CP") (footprint "Capacitor_SMD:CP_Elec_8x10")
+      (reference "C1") (unit 1) (value "22µF 16V") (footprint "Capacitor_SMD:CP_Elec_8x10")
     )
     (path "/930b2f78-333c-4610-89f3-9407fdd532f3/14be8fce-f50f-4626-ae1a-c4e73cf137a1"
@@
     )
     (path "/930b2f78-333c-4610-89f3-9407fdd532f3/258884c5-838c-4058-9ac0-9543190fd176"
-      (reference "C29") (unit 1) (value "CP") (footprint "Capacitor_SMD:CP_Elec_8x10")
+      (reference "C29") (unit 1) (value "100µF") (footprint "Capacitor_SMD:CP_Elec_8x10")
     )
     (path "/930b2f78-333c-4610-89f3-9407fdd532f3/f37548bb-87d9-41f5-9194-a353f377077f"
@@
     )
     (path "/930b2f78-333c-4610-89f3-9407fdd532f3/24fb7ed7-8d79-41c8-b99e-4c004cd9a318"
-      (reference "C35") (unit 1) (value "CP") (footprint "Capacitor_SMD:CP_Elec_8x10")
+      (reference "C35") (unit 1) (value "100µF") (footprint "Capacitor_SMD:CP_Elec_8x10")
     )
     (path "/f18cfbaa-4ca0-4a97-925e-b3011ad59682"
@@
     )
     (path "/9516bb37-bce1-45ba-96f6-12e1cc5efa7b"
-      (reference "R12") (unit 1) (value "22R") (footprint "Resistor_SMD:R_0603_1608Metric")
+      (reference "R12") (unit 1) (value "1k") (footprint "Resistor_SMD:R_0603_1608Metric")
     )
     (path "/eeb70e44-13ce-434f-85a7-b1797c59da79"

Commit message: Schematics minor changes
Other:
- note added: "Mark ON and OFF positions on the PCB Make some merkings making it obvius how to put the drivers."
Changed lines of the file:
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@@
+    (effects (font (size 1.27 1.27)) (justify left bottom))
+  )
+  (text "Mark ON and OFF positions on the PCB \nMake some merkings making it obvius how to put the drivers."
+    (at 130.81 -5.08 0)
     (effects (font (size 1.27 1.27)) (justify left bottom))
   )

Commit message: 3d model changes mostly
Other:
- note added: "Mark ON and OFF positions on the PCB Make some merkings making it obvius how to put the drivers. move console connector away from the edge"
- note removed: "Mark ON and OFF positions on the PCB Make some merkings making it obvius how to put the drivers."
Changed lines of the file:
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@@
     (effects (font (size 1.27 1.27)) (justify left bottom))
   )
-  (text "Mark ON and OFF positions on the PCB \nMake some merkings making it obvius how to put the drivers."
+  (text "Mark ON and OFF positions on the PCB \nMake some merkings making it obvius how to put the drivers.\nmove console connector away from the edge"
     (at 130.81 -5.08 0)
     (effects (font (size 1.27 1.27)) (justify left bottom))
